File: fnrow/fnrow.kicad_pcb (KiCad board)
At the start: 4 copper layers, 328.6 x 38.1 mm, 54 parts, among them J1 USB_C_Receptacle_USB2.0, J2 Conn_01x04, SW1 SW_Push, SW10 SW_Push, SW11 SW_Push, SW12 SW_Push, SW13 SW_Push, SW14 SW_Push, SW2 SW_Push, SW3 SW_Push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

Commit message: v1.2 changes
Parts:
- H1, H10, H2, H3, H4, H5, H6, H7, H8, H9: footprint MountingHole:MountingHole_2.2mm_M2 -> MountingHole:MountingHole_3.2mm_M3
- moved F1 1.55 mm to (363.4, 135.7)
- moved J1 0.46 mm to (361.4, 132.4)
Connections:
- J1 pad A8: Net-(J1-PadA8) -> unconnected-(J1-SBU1-PadA8)
- J1 pad B8: Net-(J1-PadB8) -> unconnected-(J1-SBU2-PadB8)
- U3 pad 10: Net-(U3-Pad10) -> unconnected-(U3-PA4-Pad10)
- U3 pad 11: Net-(U3-Pad11) -> unconnected-(U3-PA5-Pad11)
- U3 pad 12: Net-(U3-Pad12) -> unconnected-(U3-PA6-Pad12)
- U3 pad 13: Net-(U3-Pad13) -> unconnected-(U3-PA7-Pad13)
- U3 pad 18: Net-(U3-Pad18) -> unconnected-(U3-PA8-Pad18)
- U3 pad 19: Net-(U3-Pad19) -> unconnected-(U3-PA9-Pad19)
- U3 pad 2: Net-(U3-Pad2) -> unconnected-(U3-PF0-Pad2)
- U3 pad 20: Net-(U3-Pad20) -> unconnected-(U3-PA10-Pad20)
- U3 pad 3: Net-(U3-Pad3) -> unconnected-(U3-PF1-Pad3)
- U3 pad 31: Net-(U3-Pad31) -> unconnected-(U3-PB8-Pad31)
- U3 pad 8: Net-(U3-Pad8) -> unconnected-(U3-PA2-Pad8)
- U3 pad 9: Net-(U3-Pad9) -> unconnected-(U3-PA3-Pad9)
Routing:
- net Net-(F1-Pad2): track 14.9 -> 8.30 mm
- net +5V: track 11.3 -> 10.5 mm
- net /COL5: vias 3 -> 2
Other:
- net class Default removed
- board text added: "FnRow v1.2 12/2023 Dino Fizzotti"
- board text removed: "FnRow v1.1 12/2020 Dino Fizzotti"

Commit message: WIP
Parts:
- removed U1: LD1117S33TR_SOT223, Package_TO_SOT_SMD:SOT-223-3_TabPin2
- added C8: 100nF, Capacitor_SMD:C_0402_1005Metric, F.Cu at (357.7, 140.8)
- added U4: USBLC6-2SC6, Package_TO_SOT_SMD:SOT-23-6, F.Cu at (358.3, 138.0)
- C1: value 100nF -> 10uF; footprint Capacitor_SMD:C_0603_1608Metric_Pad1.08x0.95mm_HandSolder -> Capacitor_SMD:C_0805_2012Metric
- C2: value 10uF -> 22uF; footprint Capacitor_Tantalum_SMD:CP_EIA-3216-12_Kemet-S_Pad1.58x1.35mm_HandSolder -> Capacitor_SMD:C_0805_2012Metric
- C3: value 100nF -> 4.7uF; footprint Capacitor_SMD:C_0603_1608Metric_Pad1.08x0.95mm_HandSolder -> Capacitor_SMD:C_0603_1608Metric
- C4: value 4.7uF -> 100nF; footprint Capacitor_Tantalum_SMD:CP_EIA-3216-12_Kemet-S_Pad1.58x1.35mm_HandSolder -> Capacitor_SMD:C_0402_1005Metric
- C5, C6, C7: footprint Capacitor_SMD:C_0603_1608Metric_Pad1.08x0.95mm_HandSolder -> Capacitor_SMD:C_0402_1005Metric
- D14: footprint LED_SMD:LED_0805_2012Metric_Pad1.15x1.40mm_HandSolder -> LED_SMD:LED_0805_2012Metric
- F1: footprint Fuse:Fuse_0805_2012Metric_Pad1.15x1.40mm_HandSolder -> Fuse:Fuse_0805_2012Metric
- J1: footprint Connector_USB:USB_C_Receptacle_GCT_USB4085 -> Connector_USB:USB_C_Receptacle_HRO_TYPE-C-31-M-12
- R1, R2: footprint Resistor_SMD:R_0603_1608Metric_Pad0.98x0.95mm_HandSolder -> Capacitor_SMD:C_0402_1005Metric
- R3: value 100R -> 470R; footprint Resistor_SMD:R_0603_1608Metric_Pad0.98x0.95mm_HandSolder -> Capacitor_SMD:C_0402_1005Metric
- SW14: footprint eec:Wuerth_Elektronik-434121043816-Manufacturer_Recommended -> Button_Switch_SMD:SW_Push_1P1T_XKB_TS-1187A
- U2: value USB6B1 -> AZ1117-3.3; footprint Package_SO:SOIC-8_3.9x4.9mm_P1.27mm -> Package_TO_SOT_SMD:SOT-223
- moved C7 23.1 mm to (350.7, 134.5)
- moved C4 15.6 mm to (353.4, 150.2), turned to 180 degrees
- moved SW14 12.5 mm to (348.1, 130.8), turned to 0 degrees
- moved U2 9.38 mm to (362.8, 146.7)
- moved R2 7.97 mm to (353.9, 136.5)
- moved R1 5.24 mm to (353.9, 135.5)
- moved J1 4.56 mm to (358.3, 129.1)
- moved C5 4.44 mm to (342.0, 143.1), turned to 180 degrees
- moved C3 3.45 mm to (353.9, 151.8), turned to 180 degrees
- moved R3 3.18 mm to (341.5, 130.7), turned to 0 degrees
- moved C1 2.85 mm to (362.8, 140.8)
- moved C2 2.72 mm to (361.6, 152.3)
- moved D14 2.45 mm to (342.0, 128.9), turned to 180 degrees
- moved F1 1.76 mm to (362.8, 137.3)
- moved C6 1.27 mm to (354.7, 145.4)
Connections:
- net /COL0 renamed COL0
- net /COL1 renamed COL1
- net /COL2 renamed COL2
- net /COL3 renamed COL3
- net /COL4 renamed COL4
- net /COL5 renamed COL5
- net /COL6 renamed COL6
- net /LED renamed Net-(U3-PA15)
- net /ROW0 renamed ROW0
- net /ROW1 renamed ROW1
- net /SWCLK renamed SWCLK
- net /SWDIO renamed SWDIO
- J1 pad A6: Net-(J1-D+-PadA6) -> USB_DD+
- J1 pad A7: Net-(J1-D--PadA7) -> USB_DD-
- J1 pad B6: Net-(J1-D+-PadA6) -> USB_DD+
- J1 pad B7: Net-(J1-D--PadA7) -> USB_DD-
- U2 pad 1: +5V -> GND
- U2 pad 2: Net-(J1-D+-PadA6) -> +3V3
- U2 pad 3: Net-(J1-D--PadA7) -> +5V
- U3 pad 21: /USB_DM -> USB_D-
- U3 pad 22: /USB_DP -> USB_D+
Routing:
- net COL0: track 330.8 -> 449.3 mm, vias 2 -> 4
- net +3V3: track 375.5 -> 327.8 mm, vias 1 -> 0
- net GND: track 5.71 -> 29.4 mm, vias 3 -> 19
- net USB_D-: track 0.00 -> 23.5 mm, vias 0 -> 2
- net USB_D+: track 0.00 -> 22.2 mm, vias 0 -> 2
- net /USB_DP: track 18.9 -> 0.00 mm, vias 2 -> 0
- net /USB_DM: track 17.3 -> 0.00 mm, vias 2 -> 0
- net /NRST: track 34.7 -> 21.0 mm
- net Net-(J1-CC1): track 16.6 -> 7.20 mm, vias 0 -> 2
- net USB_DD+: track 0.00 -> 8.45 mm
- net USB_DD-: track 0.00 -> 7.73 mm, vias 0 -> 2
- net ROW0: track 310.0 -> 303.1 mm
- net Net-(J1-D--PadA7): track 5.30 -> 0.00 mm
- net Net-(J1-D+-PadA6): track 5.30 -> 0.00 mm
- net Net-(F1-Pad2): track 8.30 -> 13.2 mm
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- removed copper zone on F.Cu, net GND
Other:
- copper layers 4 -> 2
- board text added: "FnRow v1.3 12/2023 Dino Fizzotti"
- board text removed: "FnRow v1.2 12/2023 Dino Fizzotti"
